File: CameraTrigger/CameraTrigger.sch (KiCad schematic (older format))
At the start: 26 parts, among them P1 cammera_trigger_x4, P2 external_triggers, P3 analog_inputs, SW1 SW_PUSH, SW2 SW_PUSH, U1 USB, U2 AT90USB1287, U3 JTAG, X1 16MHz

Commit message: Finish preliminary layout of new motmot trigger PCB.
Parts:
- added C10: CP, symbol CP
- added P4: BNC, symbol CONN_2
Connections:
- wire segments 114 -> 119
Other:
- moved on the sheet: P1, P2, P3

Commit message: Minor corrections to boards. Labeled capacitor, etc.
Parts:
- C10: value CP -> 0.1uF
Other:
- note added: "Design by: IO Rodeo Inc."
- note added: "Released under the Creative Commons Attribution Version 3.0 License"
- note added: "http://creativecommons.org/licenses/by/3.0"
Changed lines of the file:
@@
-EESchema Schematic File Version 2  date Tue 19 Oct 2010 12:22:15 AM PDT
+EESchema Schematic File Version 2  date Wed 20 Oct 2010 07:10:42 PM PDT
 LIBS:power,/home/wbd/repos/iorodeo/CameraTriggerBoards/CameraTrigger,device,transistors,conn,linear,regul,74xx,cmos4000,adc-dac,memory,xilinx,special,microcontrollers,dsp,microchip,analog_switches,motorola,texas,intel,audio,interface,digital-audio,philips,display,cypress,siliconi,opto,atmel,contrib,valves,./CameraTrigger.cache
 EELAYER 24  0
@@
 Comment4 ""
 $EndDescr
+Text Notes 1600 7450 0    60   ~ 0
+Design by: IO Rodeo Inc.
+Text Notes 1600 7300 0    60   ~ 0
+http://creativecommons.org/licenses/by/3.0
+Text Notes 1600 7150 0    60   ~ 0
+Released under the Creative Commons Attribution Version 3.0 License
 Text Label 5950 1450 0    60   ~ 0
 GND
@@
 P 5950 1100
 F 0 "C10" H 6000 1200 50  0000 L CNN
-F 1 "CP" H 6000 1000 50  0000 L CNN
+F 1 "0.1uF" H 6000 1000 50  0000 L CNN
 	1    5950 1100
 	1    0    0    -1
