File: TriggerBreakout/TriggerBreakout.sch (KiCad schematic (older format))
At the start: 5 parts, among them P1 CONN_5X2, P2 SIGNAL_0, P3 SIGNAL_1, P4 SIGNAL_2, P5 SIGNAL_3

Commit message: Minor corrections to boards. Labeled capacitor, etc.
Other:
- note added: "Design by: Peter Polidoro, California Institute of Technology"
- note added: "Released under the Creative Commons Attribution 3.0 License"
- note added: "http://creativecommons.org/licenses/by/3.0"
- moved on the sheet: P1, P2, P3, P4, P5
Changed lines of the file:
@@
-EESchema Schematic File Version 2  date Wed 16 Jun 2010 07:01:21 PM PDT
-LIBS:power
-LIBS:device
-LIBS:transistors
-LIBS:conn
-LIBS:linear
-LIBS:regul
-LIBS:74xx
-LIBS:cmos4000
-LIBS:adc-dac
-LIBS:memory
-LIBS:xilinx
-LIBS:special
-LIBS:microcontrollers
-LIBS:dsp
-LIBS:microchip
-LIBS:analog_switches
-LIBS:motorola
-LIBS:texas
-LIBS:intel
-LIBS:audio
-LIBS:interface
-LIBS:digital-audio
-LIBS:philips
-LIBS:display
-LIBS:cypress
-LIBS:siliconi
-LIBS:opto
-LIBS:atmel
-LIBS:contrib
-LIBS:valves
-LIBS:CameraTrigger
-LIBS:TriggerBreakout-cache
+EESchema Schematic File Version 2  date Tue 19 Oct 2010 12:09:35 PM PDT
+LIBS:power,/home/wbd/repos/iorodeo/CameraTriggerBoards/CameraTrigger,device,transistors,conn,linear,regul,74xx,cmos4000,adc-dac,memory,xilinx,special,microcontrollers,dsp,microchip,analog_switches,motorola,texas,intel,audio,interface,digital-audio,philips,display,cypress,siliconi,opto,atmel,contrib,valves,./TriggerBreakout.cache
 EELAYER 24  0
 EELAYER END
@@
 Comment4 ""
 $EndDescr
-Text Label 3850 4450 0    60   ~ 0
+Text Notes 6150 6750 0    60   ~ 0
+Design by: Peter Polidoro, California Institute of Technology
+Text Notes 6150 6600 0    60   ~ 0
+http://creativecommons.org/licenses/by/3.0
+Text Notes 6150 6450 0    60   ~ 0
+Released under the Creative Commons Attribution 3.0 License
+Text Label 4950 4500 0    60   ~ 0
 Signal3
-Text Label 3850 3850 0    60   ~ 0
+Text Label 4950 3900 0    60   ~ 0
 Signal2
-Text Label 3850 3250 0    60   ~ 0
+Text Label 4950 3300 0    60   ~ 0
 Signal1
-Text Label 3850 2600 0    60   ~ 0
+Text Label 4950 2650 0    60   ~ 0
 Signal0
-Connection ~ 5100 3300
-Wire Wire Line
-	5100 3150 5100 3300
-Connection ~ 6050 3700
-Wire Wire Line
-	5950 3700 6050 3700
-Connection ~ 6050 3500
-Wire Wire Line
-	5950 3500 6050 3500
-Wire Wire Line
-	6050 3300 6050 3850
-Wire Wire Line
-	3450 3650 3550 3650
-Wire Wire Line
-	3550 3650 3550 3750
-Wire Wire Line
-	3450 2400 3550 2400
-Wire Wire Line
-	3550 2400 3550 2500
-Wire Wire Line
-	5150 3600 4450 3600
-Wire Wire Line
-	4450 3600 4450 3850
-Wire Wire Line
-	4450 3850 3450 3850
-Wire Wire Line
-	5150 3400 4650 3400
-Wire Wire Line
-	4650 3400 4650 2600
-Wire Wire Line
-	4650 2600 3450 2600
-Wire Wire Line
-	5000 3150 5000 3300
-Wire Wire Line
-	5000 3300 5150 3300
-Wire Wire Line
-	3450 3250 4550 3250
-Wire Wire Line
-	4550 3250 4550 3500
-Wire Wire Line
-	4550 3500 5150 3500
-Wire Wire Line
-	3450 4450 4550 4450
-Wire Wire Line
-	4550 4450 4550 3700
-Wire Wire Line
-	4550 3700 5150 3700
-Wire Wire Line
-	3550 3150 3550 3050
-Wire Wire Line
-	3550 3050 3450 3050
-Wire Wire Line
-	3550 4350 3550 4250
-Wire Wire Line
-	3550 4250 3450 4250
-Wire Wire Line
-	5950 3400 6050 3400
-Connection ~ 6050 3400
-Wire Wire Line
-	5950 3600 6050 3600
-Connection ~ 6050 3600
-Wire Wire Line
-	5950 3300 6200 3300
-Wire Wire Line
-	6200 3300 6200 3150
-Connection ~ 6050 3300
+Connection ~ 6200 3350
+Wire Wire Line
+	6200 3200 6200 3350
+Connection ~ 7150 3750
+Wire Wire Line
+	7050 3750 7150 3750
+Connection ~ 7150 3550
+Wire Wire Line
+	7050 3550 7150 3550
+Wire Wire Line
+	7150 3350 7150 3900
+Wire Wire Line
+	4550 3700 4650 3700
+Wire Wire Line
+	4650 3700 4650 3800
+Wire Wire Line
+	4550 2450 4650 2450
+Wire Wire Line
+	4650 2450 4650 2550
+Wire Wire Line
+	6250 3650 5550 3650
+Wire Wire Line
+	5550 3650 5550 3900
+Wire Wire Line
+	5550 3900 4550 3900
+Wire Wire Line
+	6250 3450 5750 3450
+Wire Wire Line
+	5750 3450 5750 2650
+Wire Wire Line
+	5750 2650 4550 2650
+Wire Wire Line
+	6100 3200 6100 3350
+Wire Wire Line
+	6100 3350 6250 3350
+Wire Wire Line
+	4550 3300 5650 3300
+Wire Wire Line
+	5650 3300 5650 3550
+Wire Wire Line
+	5650 3550 6250 3550
+Wire Wire Line
+	4550 4500 5650 4500
+Wire Wire Line
+	5650 4500 5650 3750
+Wire Wire Line
+	5650 3750 6250 3750
+Wire Wire Line
+	4650 3200 4650 3100
+Wire Wire Line
+	4650 3100 4550 3100
+Wire Wire Line
+	4650 4400 4650 4300
+Wire Wire Line
+	4650 4300 4550 4300
+Wire Wire Line
+	7050 3450 7150 3450
+Connection ~ 7150 3450
+Wire Wire Line
+	7050 3650 7150 3650
+Connection ~ 7150 3650
+Wire Wire Line
+	7050 3350 7300 3350
+Wire Wire Line
+	7300 3350 7300 3200
+Connection ~ 7150 3350
 $Comp
 L PWR_FLAG #FLG01
 U 1 1 4C1967A8
-P 5100 3150
-F 0 "#FLG01" H 5100 3420 30  0001 C CNN
-F 1 "PWR_FLAG" H 5100 3380 30  0000 C CNN
-	1    5100 3150
+P 6200 3200
+F 0 "#FLG01" H 6200 3470 30  0001 C CNN
+F 1 "PWR_FLAG" H 6200 3430 30  0000 C CNN
+	1    6200 3200
 	1    0    0    -1
 $EndComp
@@
 L PWR_FLAG #FLG02
 U 1 1 4C1967A0
-P 6200 3150
-F 0 "#FLG02" H 6200 3420 30  0001 C CNN
-F 1 "PWR_FLAG" H 6200 3380 30  0000 C CNN
-	1    6200 3150
+P 7300 3200
+F 0 "#FLG02" H 7300 3470 30  0001 C CNN
+F 1 "PWR_FLAG" H 7300 3430 30  0000 C CNN
+	1    7300 3200
 	1    0    0    -1
 $EndComp
@@
 L GND #PWR03
 U 1 1 4C1966FD
-P 3550 4350
-F 0 "#PWR03" H 3550 4350 30  0001 C CNN
-F 1 "GND" H 3550 4280 30  0001 C CNN
-	1    3550 4350
+P 4650 4400
+F 0 "#PWR03" H 4650 4400 30  0001 C CNN
+F 1 "GND" H 4650 4330 30  0001 C CNN
+	1    4650 4400
 	1    0    0    -1
 $EndComp
@@
 L GND #PWR04
 U 1 1 4C1966F8
-P 3550 3750
-F 0 "#PWR04" H 3550 3750 30  0001 C CNN
-F 1 "GND" H 3550 3680 30  0001 C CNN
-	1    3550 3750
+P 4650 3800
+F 0 "#PWR04" H 4650 3800 30  0001 C CNN
+F 1 "GND" H 4650 3730 30  0001 C CNN
+	1    4650 3800
 	1    0    0    -1
 $EndComp
@@
 L GND #PWR05
 U 1 1 4C1966F4
-P 3550 3150
-F 0 "#PWR05" H 3550 3150 30  0001 C CNN
-F 1 "GND" H 3550 3080 30  0001 C CNN
-	1    3550 3150
+P 4650 3200
+F 0 "#PWR05" H 4650 3200 30  0001 C CNN
+F 1 "GND" H 4650 3130 30  0001 C CNN
+	1    4650 3200
 	1    0    0    -1
 $EndComp
@@
 L GND #PWR06
 U 1 1 4C1966EF
-P 3550 2500
-F 0 "#PWR06" H 3550 2500 30  0001 C CNN
-F 1 "GND" H 3550 2430 30  0001 C CNN
-	1    3550 2500
+P 4650 2550
+F 0 "#PWR06" H 4650 2550 30  0001 C CNN
+F 1 "GND" H 4650 2480 30  0001 C CNN
+	1    4650 2550
 	1    0    0    -1
 $EndComp
@@
 L +5V #PWR07
 U 1 1 4C19667F
-P 5000 3150
-F 0 "#PWR07" H 5000 3240 20  0001 C CNN
-F 1 "+5V" H 5000 3240 30  0000 C CNN
-	1    5000 3150
+P 6100 3200
+F 0 "#PWR07" H 6100 3290 20  0001 C CNN
+F 1 "+5V" H 6100 3290 30  0000 C CNN
+	1    6100 3200
 	1    0    0    -1
 $EndComp
@@
 L GND #PWR08
 U 1 1 4C196663
-P 6050 3850
-F 0 "#PWR08" H 6050 3850 30  0001 C CNN
-F 1 "GND" H 6050 3780 30  0001 C CNN
-	1    6050 3850
+P 7150 3900
+F 0 "#PWR08" H 7150 3900 30  0001 C CNN
+F 1 "GND" H 7150 3830 30  0001 C CNN
+	1    7150 3900
 	1    0    0    -1
 $EndComp
@@
 L CONN_2 P5
 U 1 1 4C1965F0
-P 3100 4350
-F 0 "P5" V 3050 4350 40  0000 C CNN
-F 1 "SIGNAL_3" V 3150 4350 40  0000 C CNN
-	1    3100 4350
+P 4200 4400
+F 0 "P5" V 4150 4400 40  0000 C CNN
+F 1 "SIGNAL_3" V 4250 4400 40  0000 C CNN
+	1    4200 4400
 	-1   0    0    1
 $EndComp
@@
 L CONN_2 P4
 U 1 1 4C1965EE
-P 3100 3750
-F 0 "P4" V 3050 3750 40  0000 C CNN
-F 1 "SIGNAL_2" V 3150 3750 40  0000 C CNN
-	1    3100 3750
+P 4200 3800
+F 0 "P4" V 4150 3800 40  0000 C CNN
+F 1 "SIGNAL_2" V 4250 3800 40  0000 C CNN
+	1    4200 3800
 	-1   0    0    1
 $EndComp
@@
 L CONN_2 P3
 U 1 1 4C1965EB
-P 3100 3150
-F 0 "P3" V 3050 3150 40  0000 C CNN
-F 1 "SIGNAL_1" V 3150 3150 40  0000 C CNN
-	1    3100 3150
+P 4200 3200
+F 0 "P3" V 4150 3200 40  0000 C CNN
+F 1 "SIGNAL_1" V 4250 3200 40  0000 C CNN
+	1    4200 3200
 	-1   0    0    1
 $EndComp
@@
 L CONN_2 P2
 U 1 1 4C1965BD
-P 3100 2500
-F 0 "P2" V 3050 2500 40  0000 C CNN
-F 1 "SIGNAL_0" V 3150 2500 40  0000 C CNN
-	1    3100 2500
+P 4200 2550
+F 0 "P2" V 4150 2550 40  0000 C CNN
+F 1 "SIGNAL_0" V 4250 2550 40  0000 C CNN
+	1    4200 2550
 	-1   0    0    1
 $EndComp
@@
 L CONN_5X2 P1
 U 1 1 4C19655B
-P 5550 3500
-F 0 "P1" H 5550 3800 60  0000 C CNN
-F 1 "CONN_5X2" V 5550 3500 50  0000 C CNN
-	1    5550 3500
-	1    0    0    -1
-$EndComp
+P 6650 3550
+F 0 "P1" H 6650 3850 60  0000 C CNN
+F 1 "CONN_5X2" V 6650 3550 50  0000 C CNN
+	1    6650 3550
+	1    0    0    -1
+$EndComp
