File: TriggerBreakoutBuffered/TriggerBreakoutBuffered.sch (KiCad schematic (older format))
At the start: 7 parts, among them P1 CONN_5X2, P2 SIGNAL_0, P3 SIGNAL_1, P4 SIGNAL_2, P5 SIGNAL_3, U1 74LS125

Commit message: Minor corrections to boards. Labeled capacitor, etc.
Other:
- note added: "Design by: Peter Polidoro, California Institute of Technology"
- note added: "Released under the Creative Commons Attribution 3.0 License"
- note added: "http://creativecommons.org/license/by/3.0"
- moved on the sheet: C1, P1, P2, P3, P4, P5, U1A, U1B, U1C, U1D
